File: eagle/TFTbarebones.sch (EAGLE design)
At the start: 18 parts, among them IC5 APX803, Q1 MMBT2222, U2 MIC5225-3.3, U3 74HC4050D

Commit message: mini probe
Parts:
- removed C1, C2: 10µF, microbuilder:CAP_CERAMIC0805-NOOUTLINE
- removed C3: 0.1uF, microbuilder:CAP_CERAMIC0805-NOOUTLINE
- removed CN1: (no value), microbuilder:MICROSD
- removed FID1, FID2: FIDUCIAL_1MM, microbuilder:FIDUCIAL_1MM
- removed Q1: MMBT2222, microbuilder:TRANSISTOR_NPNWIDE
- removed R7: 1K, microbuilder:RESISTOR_0603_NOOUT
- removed R8: 10K, microbuilder:RESISTOR_0603_NOOUT
- removed U2: MIC5225-3.3, microbuilder:VREG_SOT23-5
- removed U3: 74HC4050D, microbuilder:74HC4050D
Connections:
- removed net !TFTRST_3V: DISP1.RESET, U3.5Y
- removed net 3.3V: C1.1, C3.1, CN1.SD_VDD, DISP1.LEDA, DISP1.VDD, IC5.VCC, JP1.2, R2.2, R8.2, U2.OUT, U3.VCC
- removed net BACKLIGHT: JP1.11, R7.1, R8.1
- removed net DC_3V: DISP1.RS/DC, U3.6Y
- removed net MISO_3V: CN1.DATA_OUT, JP1.5
- removed net MOSI_3V: CN1.DATA_IN, DISP1.DATA, U3.3Y
- removed net N$1: Q1.B, R7.2
- removed net N$5: Q1.C, R5.1
- removed net SCK_3V: CN1.SCLK, DISP1.CLOCK, U3.2Y
- removed net SDCS: JP1.10, U3.4A
- removed net SDCS_3V: CN1.CS, U3.4Y
- removed net TFTCS_3V: DISP1.CS, U3.1Y
- removed net VIN: C2.1, JP1.1, U2.EN, U2.IN
- new net 3V: DISP1.LEDA, DISP1.VDD, IC5.VCC, JP1.2, R2.2
- net !TFTRST: now also DISP1.RESET; no longer U3.5A
- net DC: now also DISP1.RS/DC; no longer U3.6A
- net GND: now also R5.1; no longer C1.2, C2.2, C3.2, CN1.GND@1, CN1.GND@2, CN1.GND@3, Q1.E, U2.GND, U3.GND
- net MOSI: now also DISP1.DATA; no longer U3.3A
- net SCK: now also DISP1.CLOCK; no longer U3.2A
- net TFTCS: now also DISP1.CS; no longer U3.1A
Other:
- moved on the sheet: IC5, JP1, R2, R5
