File: eagle/probe20mm.brd (EAGLE design)
At the start: 20 x 20 mm, 8 parts

Commit message: mini probe
Routing:
- net N$1: track 46.3 -> 0.00 mm
- net N$2: track 45.3 -> 0.00 mm
- net N$4: track 43.4 -> 0.00 mm
- net REAR: track 4.33 -> 0.00 mm, vias 2 -> 0
- net FACE: track 1.31 -> 0.00 mm, vias 1 -> 0

Commit message: mini probe redesign
Parts:
- moved FACE 3.88 mm to (10.2, 16.2)
- moved REAR 2.24 mm to (7.00, 18.0)
Routing:
- net N$1: track 0.00 -> 60.2 mm
- net N$2: track 0.00 -> 37.2 mm
- net N$4: track 0.00 -> 33.8 mm
- net FACE: track 0.00 -> 1.41 mm, vias 0 -> 1

Commit message: probe base
Parts:
- removed REAR: TPTP10R, testpad:TP10R
- added R1: 10k, resistor:R0805
- added U1: MLX90614ESF-BAA-000-TU, MLX90614ESF-BAA-000-TU:TO254P942H425-4
- FACE: value TPTP10R -> TPTP14R; device testpad:TP10R -> testpad:TP14R
- moved FACE 1.22 mm to (10.0, 15.0)
Connections:
- removed net N$1: TO1.A, TO2.A, TO3.A, UV1.A, UV2.A, UV3.A
- removed net REAR: REAR.TP
- new net 3V: R1.2, TO1.A, TO2.A, TO3.A, U1.3, UV1.A, UV2.A, UV3.A
- new net GND: U1.4
- new net SCL: R1.1, U1.1
Routing:
- net 3V: track 0.00 -> 67.0 mm
- net N$1: track 60.2 -> 0.00 mm
- net N$4: track 33.8 -> 26.1 mm
- net N$2: track 37.2 -> 43.5 mm
- net SCL: track 0.00 -> 1.59 mm
- added copper zone on layer 1, net GND
- removed copper zone on layer 1, net REAR
Other:
- board text added: "3V"
- board text added: "GND"
- board text added: "SCL"
- board text added: "SDA/PWM"
