File: eagle/probe20mm.sch (EAGLE design)
At the start: 8 parts

Commit message: probe base
Parts:
- removed REAR: TPTP10R, testpad:TPTP10R
- added R1: 10k, resistor:R-EU_R0805
- added U1: MLX90614ESF-BAA-000-TU, MLX90614ESF-BAA-000-TU:MLX90614ESF-BAA-000-TU
- FACE: value TPTP10R -> TPTP14R; device testpad:TPTP10R -> testpad:TPTP14R
Connections:
- removed net N$1: TO1.A, TO2.A, TO3.A, UV1.A, UV2.A, UV3.A
- removed net REAR: REAR.TP
- new net 3V: R1.2, TO1.A, TO2.A, TO3.A, U1.VDD, UV1.A, UV2.A, UV3.A
- new net GND: U1.VSS
- new net SCL: R1.1, U1.SCL/VZ
Changed lines of the file:
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@@
 <part name="UV2" library="general" deviceset="LED" device="5MM" package3d_urn="urn:adsk.eagle:package:15799/2"/>
 <part name="UV3" library="general" deviceset="LED" device="5MM" package3d_urn="urn:adsk.eagle:package:15799/2"/>
-<part name="FACE" library="testpad" library_urn="urn:adsk.eagle:library:385" deviceset="TP" device="TP10R" package3d_urn="urn:adsk.eagle:package:27959/1"/>
-<part name="REAR" library="testpad" library_urn="urn:adsk.eagle:library:385" deviceset="TP" device="TP10R" package3d_urn="urn:adsk.eagle:package:27959/1"/>
+<part name="U1" library="MLX90614ESF-BAA-000-TU" deviceset="MLX90614ESF-BAA-000-TU" device=""/>
+<part name="FACE" library="testpad" library_urn="urn:adsk.eagle:library:385" deviceset="TP" device="TP14R" package3d_urn="urn:adsk.eagle:package:27966/1"/>
+<part name="R1" library="resistor" library_urn="urn:adsk.eagle:library:348" deviceset="R-EU_" device="R0805" package3d_urn="urn:adsk.eagle:package:23553/2" value="10k"/>
 </parts>
 <sheets>
@@
 <attribute name="VALUE" x="43.815" y="46.228" size="1.778" layer="96" rot="R90"/>
 </instance>
+<instance part="U1" gate="G$1" x="2.54" y="33.02" smashed="yes">
+<attribute name="NAME" x="-7.62" y="39.37" size="1.778" layer="95"/>
+<attribute name="VALUE" x="-7.62" y="22.86" size="1.778" layer="96"/>
+</instance>
 <instance part="FACE" gate="G$1" x="50.8" y="55.88" smashed="yes">
 <attribute name="NAME" x="49.53" y="57.15" size="1.778" layer="95"/>
 <attribute name="TP_SIGNAL_NAME" x="52.07" y="54.61" size="1.778" layer="97"/>
 </instance>
-<instance part="REAR" gate="G$1" x="58.42" y="55.88" smashed="yes">
-<attribute name="NAME" x="57.15" y="57.15" size="1.778" layer="95"/>
-<attribute name="TP_SIGNAL_NAME" x="59.69" y="54.61" size="1.778" layer="97"/>
+<instance part="R1" gate="G$1" x="2.54" y="43.18" smashed="yes">
+<attribute name="NAME" x="-1.27" y="44.6786" size="1.778" layer="95"/>
+<attribute name="VALUE" x="-1.27" y="39.878" size="1.778" layer="96"/>
 </instance>
 </instances>
@@
 </busses>
 <nets>
-<net name="N$1" class="0">
-<segment>
-<pinref part="TO1" gate="G$1" pin="A"/>
-<pinref part="TO2" gate="G$1" pin="A"/>
-<wire x1="-30.48" y1="53.34" x2="-22.86" y2="53.34" width="0.1524" layer="91"/>
-<pinref part="TO3" gate="G$1" pin="A"/>
-<wire x1="-22.86" y1="53.34" x2="-15.24" y2="53.34" width="0.1524" layer="91"/>
-<junction x="-22.86" y="53.34"/>
-<junction x="-15.24" y="53.34"/>
-<pinref part="UV1" gate="G$1" pin="A"/>
-<pinref part="UV2" gate="G$1" pin="A"/>
-<wire x1="22.86" y1="53.34" x2="30.48" y2="53.34" width="0.1524" layer="91"/>
-<pinref part="UV3" gate="G$1" pin="A"/>
-<wire x1="30.48" y1="53.34" x2="38.1" y2="53.34" width="0.1524" layer="91"/>
-<junction x="30.48" y="53.34"/>
-<wire x1="-15.24" y1="53.34" x2="22.86" y2="53.34" width="0.1524" layer="91"/>
-<junction x="22.86" y="53.34"/>
-</segment>
-</net>
 <net name="N$2" class="0">
 <segment>
@@
 <net name="FACE" class="0">
 <segment>
-<pinref part="FACE" gate="G$1" pin="TP"/>
 <wire x1="50.8" y1="53.34" x2="50.8" y2="45.72" width="0.1524" layer="91"/>
 <label x="47.498" y="43.688" size="1.778" layer="95"/>
+<pinref part="FACE" gate="G$1" pin="TP"/>
 </segment>
 </net>
-<net name="REAR" class="0">
+<net name="GND" class="0">
 <segment>
-<pinref part="REAR" gate="G$1" pin="TP"/>
-<wire x1="58.42" y1="53.34" x2="58.42" y2="45.72" width="0.1524" layer="91"/>
-<label x="55.118" y="43.688" size="1.778" layer="95"/>
+<pinref part="U1" gate="G$1" pin="VSS"/>
+<wire x1="17.78" y1="27.94" x2="25.4" y2="27.94" width="0.1524" layer="91"/>
+<label x="25.4" y="27.94" size="1.778" layer="95"/>
 </segment>
 </net>
+<net name="3V" class="0">
+<segment>
+<pinref part="U1" gate="G$1" pin="VDD"/>
+<wire x1="17.78" y1="35.56" x2="20.32" y2="35.56" width="0.1524" layer="91"/>
+<label x="25.4" y="35.56" size="1.778" layer="95"/>
+<pinref part="R1" gate="G$1" pin="2"/>
+<wire x1="20.32" y1="35.56" x2="25.4" y2="35.56" width="0.1524" layer="91"/>
+<wire x1="7.62" y1="43.18" x2="20.32" y2="43.18" width="0.1524" layer="91"/>
+<wire x1="20.32" y1="43.18" x2="20.32" y2="35.56" width="0.1524" layer="91"/>
+<junction x="20.32" y="35.56"/>
+</segment>
+<segment>
+<pinref part="TO1" gate="G$1" pin="A"/>
+<pinref part="TO2" gate="G$1" pin="A"/>
+<wire x1="-30.48" y1="53.34" x2="-22.86" y2="53.34" width="0.1524" layer="91"/>
+<pinref part="TO3" gate="G$1" pin="A"/>
+<wire x1="-22.86" y1="53.34" x2="-15.24" y2="53.34" width="0.1524" layer="91"/>
+<junction x="-22.86" y="53.34"/>
+<junction x="-15.24" y="53.34"/>
+<pinref part="UV1" gate="G$1" pin="A"/>
+<pinref part="UV2" gate="G$1" pin="A"/>
+<wire x1="22.86" y1="53.34" x2="30.48" y2="53.34" width="0.1524" layer="91"/>
+<pinref part="UV3" gate="G$1" pin="A"/>
+<wire x1="30.48" y1="53.34" x2="38.1" y2="53.34" width="0.1524" layer="91"/>
+<junction x="30.48" y="53.34"/>
+<wire x1="-15.24" y1="53.34" x2="22.86" y2="53.34" width="0.1524" layer="91"/>
+<junction x="22.86" y="53.34"/>
+</segment>
+</net>
+<net name="SCL" class="0">
+<segment>
+<pinref part="U1" gate="G$1" pin="SCL/VZ"/>
+<wire x1="-12.7" y1="33.02" x2="-12.7" y2="43.18" width="0.1524" layer="91"/>
+<pinref part="R1" gate="G$1" pin="1"/>
+<wire x1="-12.7" y1="43.18" x2="-2.54" y2="43.18" width="0.1524" layer="91"/>
+</segment>
+</net>
