File: eagle/probebase.brd (EAGLE design)
At the start: 18.5 x 16 mm, 17 parts, among them IC5 APX803

Commit message: misc pcb changes
Changed lines of the file:
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@@
 <wire x1="10" y1="8.5" x2="10.54" y2="7.96" width="0.1524" layer="16"/>
 <wire x1="10.54" y1="7.96" x2="13.43" y2="7.96" width="0.1524" layer="16"/>
-<wire x1="2.5" y1="7.75" x2="2.6214" y2="7.8714" width="0.1524" layer="16"/>
-<wire x1="2.6214" y1="7.8714" x2="3.3446875" y2="7.8714" width="0.1524" layer="16"/>
-<wire x1="3.3446875" y1="7.8714" x2="3.4184875" y2="7.9452" width="0.1524" layer="16"/>
 <wire x1="8.320925" y1="7.24801875" x2="8.320925" y2="6.820925" width="0.1524" layer="16"/>
 <wire x1="3.4184875" y1="7.9452" x2="7.62374375" y2="7.9452" width="0.1524" layer="16"/>
 <wire x1="7.62374375" y1="7.9452" x2="8.320925" y2="7.24801875" width="0.1524" layer="16"/>
+<wire x1="2.5" y1="7.75" x2="3.2232875" y2="7.75" width="0.1524" layer="16"/>
+<wire x1="3.2232875" y1="7.75" x2="3.4184875" y2="7.9452" width="0.1524" layer="16"/>
 </signal>
 <signal name="TFTRST">
@@
 <wire x1="2.5" y1="6.25" x2="4.81894375" y2="6.25" width="0.1524" layer="16"/>
 <wire x1="14.50094375" y1="3.0516" x2="14.8134" y2="3.36405625" width="0.1524" layer="16"/>
-<wire x1="14.3746875" y1="6.9636" x2="13.7264" y2="6.9636" width="0.1524" layer="16"/>
-<wire x1="13.7264" y1="6.9636" x2="13.43" y2="7.26" width="0.1524" layer="16"/>
-<wire x1="14.8134" y1="3.36405625" x2="14.8134" y2="6.5248875" width="0.1524" layer="16"/>
-<wire x1="14.8134" y1="6.5248875" x2="14.3746875" y2="6.9636" width="0.1524" layer="16"/>
+<wire x1="14.8134" y1="6.5248875" x2="14.8134" y2="3.36405625" width="0.1524" layer="16"/>
 <wire x1="4.81894375" y1="6.25" x2="8.01734375" y2="3.0516" width="0.1524" layer="16"/>
 <wire x1="8.01734375" y1="3.0516" x2="14.50094375" y2="3.0516" width="0.1524" layer="16"/>
+<wire x1="13.43" y1="7.26" x2="14.0782875" y2="7.26" width="0.1524" layer="16"/>
+<wire x1="14.0782875" y1="7.26" x2="14.8134" y2="6.5248875" width="0.1524" layer="16"/>
 </signal>
 <signal name="DC">
@@
 <contactref element="U$3" pad="7"/>
 <wire x1="14.3746875" y1="3.3564" x2="14.5086" y2="3.4903125" width="0.1524" layer="16"/>
-<wire x1="14.5086" y1="6.1296875" x2="14.3746875" y2="6.2636" width="0.1524" layer="16"/>
-<wire x1="14.3746875" y1="6.2636" x2="13.7264" y2="6.2636" width="0.1524" layer="16"/>
-<wire x1="14.5086" y1="3.4903125" x2="14.5086" y2="6.1296875" width="0.1524" layer="16"/>
-<wire x1="13.7264" y1="6.2636" x2="13.43" y2="6.56" width="0.1524" layer="16"/>
+<wire x1="14.5086" y1="6.1296875" x2="14.5086" y2="3.4903125" width="0.1524" layer="16"/>
 <wire x1="8.1436" y1="3.3564" x2="14.3746875" y2="3.3564" width="0.1524" layer="16"/>
-<wire x1="2.5" y1="7.25" x2="2.6214" y2="7.1286" width="0.1524" layer="16"/>
-<wire x1="2.6214" y1="7.1286" x2="3.3446875" y2="7.1286" width="0.1524" layer="16"/>
-<wire x1="3.3446875" y1="7.1286" x2="3.9184875" y2="6.5548" width="0.1524" layer="16"/>
 <wire x1="4.9452" y1="6.5548" x2="8.1436" y2="3.3564" width="0.1524" layer="16"/>
 <wire x1="3.9184875" y1="6.5548" x2="4.9452" y2="6.5548" width="0.1524" layer="16"/>
+<wire x1="13.43" y1="6.56" x2="14.0782875" y2="6.56" width="0.1524" layer="16"/>
+<wire x1="14.0782875" y1="6.56" x2="14.5086" y2="6.1296875" width="0.1524" layer="16"/>
+<wire x1="2.5" y1="7.25" x2="3.2232875" y2="7.25" width="0.1524" layer="16"/>
+<wire x1="3.2232875" y1="7.25" x2="3.9184875" y2="6.5548" width="0.1524" layer="16"/>
 </signal>
 <signal name="SCK">
 <contactref element="U$4" pad="4"/>
 <contactref element="U$3" pad="10"/>
-<wire x1="2.5" y1="8.75" x2="2.6214" y2="8.6286" width="0.1524" layer="16"/>
-<wire x1="2.6214" y1="8.6286" x2="3.3446875" y2="8.6286" width="0.1524" layer="16"/>
-<wire x1="3.3446875" y1="8.6286" x2="3.4184875" y2="8.5548" width="0.1524" layer="16"/>
-<wire x1="12.3865125" y1="5.4648" x2="12.4853125" y2="5.5636" width="0.1524" layer="16"/>
-<wire x1="12.4853125" y1="5.5636" x2="13.1336" y2="5.5636" width="0.1524" layer="16"/>
-<wire x1="13.1336" y1="5.5636" x2="13.43" y2="5.86" width="0.1524" layer="16"/>
 <wire x1="3.4184875" y1="8.5548" x2="7.87625625" y2="8.5548" width="0.1524" layer="16"/>
 <wire x1="7.87625625" y1="8.5548" x2="10.96625625" y2="5.4648" width="0.1524" layer="16"/>
-<wire x1="10.96625625" y1="5.4648" x2="12.3865125" y2="5.4648" width="0.1524" layer="16"/>
+<wire x1="12.3865125" y1="5.4648" x2="10.96625625" y2="5.4648" width="0.1524" layer="16"/>
+<wire x1="13.43" y1="5.86" x2="12.7817125" y2="5.86" width="0.1524" layer="16"/>
+<wire x1="12.7817125" y1="5.86" x2="12.3865125" y2="5.4648" width="0.1524" layer="16"/>
+<wire x1="2.5" y1="8.75" x2="3.2232875" y2="8.75" width="0.1524" layer="16"/>
+<wire x1="3.2232875" y1="8.75" x2="3.4184875" y2="8.5548" width="0.1524" layer="16"/>
 </signal>
 <signal name="MOSI">
@@
 <wire x1="0.7084" y1="2.2916" x2="0.7084" y2="2.5" width="0.1524" layer="1"/>
 <via x="0.7084" y="2.5" extent="1-16" drill="0.35"/>
-<wire x1="0.7084" y1="2.5" x2="2.4584" y2="4.25" width="0.1524" layer="16"/>
-<wire x1="2.4584" y1="4.25" x2="2.5" y2="4.25" width="0.1524" layer="16"/>
+<wire x1="2.5" y1="4.25" x2="1.75" y2="4.25" width="0.1524" layer="16"/>
+<wire x1="0.7084" y1="3.2084" x2="0.7084" y2="2.5" width="0.1524" layer="16"/>
+<wire x1="1.75" y1="4.25" x2="0.7084" y2="3.2084" width="0.1524" layer="16"/>
 </signal>
 <signal name="L2-">
@@
 <wire x1="4" y1="3" x2="3" y2="2" width="0.1524" layer="1"/>
 <via x="3" y="2" extent="1-16" drill="0.35"/>
-<wire x1="3.4786" y1="4.0053125" x2="3.4786" y2="4.4946875" width="0.1524" layer="16"/>
-<wire x1="3.4786" y1="4.4946875" x2="3.3446875" y2="4.6286" width="0.1524" layer="16"/>
-<wire x1="3.3446875" y1="4.6286" x2="2.6214" y2="4.6286" width="0.1524" layer="16"/>
-<wire x1="2.6214" y1="4.6286" x2="2.5" y2="4.75" width="0.1524" layer="16"/>
+<wire x1="3.4786" y1="4.4946875" x2="3.4786" y2="4.0053125" width="0.1524" layer="16"/>
 <wire x1="3" y1="2" x2="3" y2="3.5267125" width="0.1524" layer="16"/>
 <wire x1="3" y1="3.5267125" x2="3.4786" y2="4.0053125" width="0.1524" layer="16"/>
+<wire x1="2.5" y1="4.75" x2="3.2232875" y2="4.75" width="0.1524" layer="16"/>
+<wire x1="3.2232875" y1="4.75" x2="3.4786" y2="4.4946875" width="0.1524" layer="16"/>
 </signal>
 <signal name="L3-">
@@
 <wire x1="4" y1="5.5" x2="5" y2="4.5" width="0.1524" layer="1"/>
 <via x="5" y="4.5" extent="1-16" drill="0.35"/>
-<wire x1="3.3446875" y1="5.6286" x2="2.6214" y2="5.6286" width="0.1524" layer="16"/>
-<wire x1="2.6214" y1="5.6286" x2="2.5" y2="5.75" width="0.1524" layer="16"/>
-<wire x1="5" y1="4.5" x2="4.4732875" y2="4.5" width="0.1524" layer="16"/>
-<wire x1="4.4732875" y1="4.5" x2="3.3446875" y2="5.6286" width="0.1524" layer="16"/>
+<wire x1="4.4732875" y1="4.5" x2="5" y2="4.5" width="0.1524" layer="16"/>
+<wire x1="2.5" y1="5.75" x2="3.2232875" y2="5.75" width="0.1524" layer="16"/>
+<wire x1="3.2232875" y1="5.75" x2="4.4732875" y2="4.5" width="0.1524" layer="16"/>
 </signal>
 <signal name="SDA">
@@
 <wire x1="4" y1="8.5" x2="5.5" y2="10" width="0.1524" layer="1"/>
 <via x="5.5" y="10" extent="1-16" drill="0.35"/>
-<wire x1="3.3446875" y1="9.3714" x2="2.6214" y2="9.3714" width="0.1524" layer="16"/>
-<wire x1="2.6214" y1="9.3714" x2="2.5" y2="9.25" width="0.1524" layer="16"/>
-<wire x1="5.5" y1="10" x2="3.9732875" y2="10" width="0.1524" layer="16"/>
-<wire x1="3.9732875" y1="10" x2="3.3446875" y2="9.3714" width="0.1524" layer="16"/>
+<wire x1="3.9732875" y1="10" x2="5.5" y2="10" width="0.1524" layer="16"/>
+<wire x1="2.5" y1="9.25" x2="3.2232875" y2="9.25" width="0.1524" layer="16"/>
+<wire x1="3.2232875" y1="9.25" x2="3.9732875" y2="10" width="0.1524" layer="16"/>
 </signal>
 <signal name="SCL">
@@
 <wire x1="4" y1="10.5" x2="5" y2="11.5" width="0.1524" layer="1"/>
 <via x="5" y="11.5" extent="1-16" drill="0.35"/>
-<wire x1="3.3446875" y1="10.3714" x2="2.6214" y2="10.3714" width="0.1524" layer="16"/>
-<wire x1="2.6214" y1="10.3714" x2="2.5" y2="10.25" width="0.1524" layer="16"/>
-<wire x1="5" y1="11.5" x2="4.4732875" y2="11.5" width="0.1524" layer="16"/>
-<wire x1="4.4732875" y1="11.5" x2="3.3446875" y2="10.3714" width="0.1524" layer="16"/>
+<wire x1="4.4732875" y1="11.5" x2="5" y2="11.5" width="0.1524" layer="16"/>
+<wire x1="2.5" y1="10.25" x2="3.2232875" y2="10.25" width="0.1524" layer="16"/>
+<wire x1="3.2232875" y1="10.25" x2="4.4732875" y2="11.5" width="0.1524" layer="16"/>
 </signal>
 <signal name="BCLK">
@@
 <wire x1="3.5" y1="13.5" x2="3.5" y2="14.5" width="0.1524" layer="1"/>
 <via x="3.5" y="14.5" extent="1-16" drill="0.35"/>
-<wire x1="3.5" y1="14.5" x2="2.5" y2="13.5" width="0.1524" layer="16"/>
-<wire x1="2.5" y1="13.5" x2="2.5" y2="11.75" width="0.1524" layer="16"/>
+<wire x1="3.5" y1="14.5" x2="3.5" y2="12" width="0.1524" layer="16"/>
+<wire x1="3.5" y1="12" x2="3.25" y2="11.75" width="0.1524" layer="16"/>
+<wire x1="3.25" y1="11.75" x2="2.5" y2="11.75" width="0.1524" layer="16"/>
 </signal>
 </signals>
